Commit message: default - black color

File: turtlebot1_descriptions/roomba_description/urdf/roomba.urdf.xacro (robot description, xacro)
@@ -38,6 +38,6 @@
 	    	<visual>
 	      		<origin xyz=" 0 0 0.0308" rpy="0 0 1.5708" />
-	      		<geometry>
-	        		<mesh filename="package://roomba_description/meshes/$(arg color)_roomba.dae"/>
+                        <geometry>  <!-- roomba color set to black in 20.setup.bash.em-->
+                                <mesh filename="package://roomba_description/meshes/$(env ROOMBA_COLOR)_roomba.dae"/>
 	      		</geometry>
 	    	</visual>

Commit message: adapted so that it will also work under ros-kinetic

File: turtlebot1_descriptions/roomba_description/urdf/roomba.urdf.xacro (robot description, xacro)
@@ -6,4 +6,5 @@
       <alwaysOn>true</alwaysOn>
       <updateRate>40</updateRate>
+      <legacyMode>false</legacyMode>
       <leftJoint>left_wheel_joint</leftJoint>
       <rightJoint>right_wheel_joint</rightJoint>
@@ -25,5 +26,5 @@
 	      		<origin xyz="0 0 0" rpy="0 0 0" />
 	      		<geometry>
-	        		<cylinder length="0" radius="0.16495"/>
+                                <cylinder length="0.001" radius="0.16495"/>
 	     	 	</geometry>
 	    	</collision>

Commit message: minor changes

File: turtlebot1_descriptions/roomba_description/urdf/roomba.urdf.xacro (robot description, xacro)
@@ -26,5 +26,5 @@
 	      		<origin xyz="0 0 0" rpy="0 0 0" />
 	      		<geometry>
-                                <cylinder length="0.001" radius="0.16495"/>
+                                cd <cylinder length="0.001" radius="0.16495"/>
 	     	 	</geometry>
 	    	</collision>
